Commit message: motor driver

File: agv_hw/urdf/ros2_control.xacro (robot description, xacro)
@@ -1,25 +1,19 @@
 <?xml version="1.0"?>
 <robot xmlns:xacro="http://www.ros.org/wiki/xacro">
-    <ros2_control name="AGV" type="actuator">
+    <ros2_control name="AGV" type="system">
         <hardware>
-            <plugin>agv_hw/Robomaster6020</plugin>
+            <plugin>agv_hw/Tiger_motor</plugin>
             <param name="can_name">can0</param>
-            <param name="motor_id">1</param>
+            <param name="motor_id_left">1</param>
+            <param name="motor_id_right">2</param>
         </hardware>
         <joint name="left_wheel_joint">
-            <command_interface name="effort"/>
-            <state_interface name="effort"/>
-            <state_interface name="velocity"/>
+            <command_interface name="velocity"/>
             <state_interface name="position"/>
-            <state_interface name="temperature"/>
         </joint>
-        <!-- <joint name="right_wheel_joint">
-            <command_interface name="velocity">
-                <param name="min">-10</param>
-                <param name="max">10</param>
-            </command_interface>
-            <state_interface name="velocity"/>
+        <joint name="right_wheel_joint">
+            <command_interface name="velocity"/>
             <state_interface name="position"/>
-        </joint> -->
+        </joint>
     </ros2_control>
 </robot>
