Commit message: agv.dae

File: agv_description/urdf/body.xacro (robot description, xacro)
@@ -11,11 +11,13 @@
     <link name="chassis">
         <visual>
-            <origin xyz="0 0 0.4"/>
+            <!-- <origin xyz="0 0 0.4"/> -->
+            <!-- <pose>0 0 0 0 0 0</pose> -->
             <geometry>
-                <box size="1 0.52 0.7"/>
+                <mesh filename="package://agv_description/mesh/agv.dae"/>
+                <scale>0.0001 0.0001 0.0001</scale>
             </geometry>
             <material name="white"/>
         </visual>
-        <collision>
+        <!-- <collision>
             <origin xyz="0 0 0.4"/>
             <geometry>
@@ -25,5 +27,5 @@
         <xacro:inertial_box mass="10" x="1" y="0.52" z="0.7">
             <origin xyz="0 0 0.4" rpy="0 0 0"/>
-        </xacro:inertial_box>
+        </xacro:inertial_box> -->
     </link>
     <!-- LEFT WHEEL -->

Commit message: add body.stl

File: agv_description/urdf/body.xacro (robot description, xacro)
@@ -11,13 +11,11 @@
     <link name="chassis">
         <visual>
-            <!-- <origin xyz="0 0 0.4"/> -->
-            <!-- <pose>0 0 0 0 0 0</pose> -->
+            <origin xyz="-0.4 -0.26 0"/>
             <geometry>
-                <mesh filename="package://agv_description/mesh/agv.dae"/>
-                <scale>0.0001 0.0001 0.0001</scale>
+                <mesh filename="package://agv_description/meshes/body.stl" scale="0.001 0.001 0.001"/>
             </geometry>
             <material name="white"/>
         </visual>
-        <!-- <collision>
+        <collision>
             <origin xyz="0 0 0.4"/>
             <geometry>
@@ -27,5 +25,5 @@
         <xacro:inertial_box mass="10" x="1" y="0.52" z="0.7">
             <origin xyz="0 0 0.4" rpy="0 0 0"/>
-        </xacro:inertial_box> -->
+        </xacro:inertial_box>
     </link>
     <!-- LEFT WHEEL -->

Commit message: agv_look_color

File: agv_description/urdf/body.xacro (robot description, xacro)
@@ -9,13 +9,23 @@
         <origin xyz="0 0 0"/>
     </joint>
+    <joint name="gaizi_front_joint" type="fixed">
+        <parent link="base_link"/>
+        <child link="gaizi_front"/>
+        <origin xyz="0 0 0"/>
+    </joint>
+    <joint name="gaizi_back_joint" type="fixed">
+        <parent link="base_link"/>
+        <child link="gaizi_back"/>
+        <origin xyz="0 0 0"/>
+    </joint>
     <link name="chassis">
         <visual>
-            <origin xyz="-0.4 -0.26 0"/>
+            <origin xyz="0 0 0" rpy="0 0 0" />
             <geometry>
-                <mesh filename="package://agv_description/meshes/body.stl" scale="0.001 0.001 0.001"/>
+                <mesh filename="package://agv_description/meshes/chassis.stl" scale ="0.001 0.001 0.001"/>
             </geometry>
             <material name="white"/>
         </visual>
-        <collision>
+        <!-- <collision>
             <origin xyz="0 0 0.4"/>
             <geometry>
@@ -25,5 +35,29 @@
         <xacro:inertial_box mass="10" x="1" y="0.52" z="0.7">
             <origin xyz="0 0 0.4" rpy="0 0 0"/>
-        </xacro:inertial_box>
+        </xacro:inertial_box> -->
+    </link>
+    <!-- gaizi_front -->
+    <link name="gaizi_front">
+        <visual>
+            <origin xyz="0 0 0" rpy="0 0 0" />
+            <geometry>
+                <mesh filename="package://agv_description/meshes/gaizi.stl" scale ="0.001 0.001 0.001"/>
+            </geometry>
+            <material name="orange">
+                <color rgba="1.0 0.4235 0.0392 1.0"/>
+            </material>
+        </visual>
+    </link>
+    <!-- gaizi_back -->
+    <link name="gaizi_back">
+        <visual>
+            <origin xyz="0 0 0" rpy="0 0 ${pi}" />
+            <geometry>
+                <mesh filename="package://agv_description/meshes/gaizi.stl" scale ="0.001 0.001 0.001"/>
+            </geometry>
+            <material name="orange">
+                <color rgba="1.0 0.4235 0.0392 1.0"/>
+            </material>
+        </visual>
     </link>
     <!-- LEFT WHEEL -->

Commit message: gazebo show stl

File: agv_description/urdf/body.xacro (robot description, xacro)
@@ -23,5 +23,6 @@
             <origin xyz="0 0 0" rpy="0 0 0" />
             <geometry>
-                <mesh filename="package://agv_description/meshes/chassis.stl" scale ="0.001 0.001 0.001"/>
+                <!-- <mesh filename="package://agv_description/meshes/chassis.stl" scale ="0.001 0.001 0.001"/> -->
+                <mesh filename="/home/cc/.gazebo/models/chassis.stl" scale ="0.001 0.001 0.001"/>
             </geometry>
             <material name="white"/>
@@ -42,5 +43,6 @@
             <origin xyz="0 0 0" rpy="0 0 0" />
             <geometry>
-                <mesh filename="package://agv_description/meshes/gaizi.stl" scale ="0.001 0.001 0.001"/>
+                <!-- <mesh filename="package://agv_description/meshes/gaizi.stl" scale ="0.001 0.001 0.001"/> -->
+                <mesh filename="/home/cc/.gazebo/models/gaizi.stl" scale ="0.001 0.001 0.001"/>
             </geometry>
             <material name="orange">
@@ -49,4 +51,7 @@
         </visual>
     </link>
+    <gazebo reference="gaizi_front">
+	    <material>Gazebo/Orange</material>
+    </gazebo>
     <!-- gaizi_back -->
     <link name="gaizi_back">
@@ -54,5 +59,6 @@
             <origin xyz="0 0 0" rpy="0 0 ${pi}" />
             <geometry>
-                <mesh filename="package://agv_description/meshes/gaizi.stl" scale ="0.001 0.001 0.001"/>
+                <!-- <mesh filename="package://agv_description/meshes/gaizi.stl" scale ="0.001 0.001 0.001"/> -->
+                <mesh filename="/home/cc/.gazebo/models/gaizi.stl" scale ="0.001 0.001 0.001"/>
             </geometry>
             <material name="orange">
@@ -61,4 +67,7 @@
         </visual>
     </link>
+    <gazebo reference="gaizi_back">
+	    <material>Gazebo/Orange</material>
+    </gazebo>
     <!-- LEFT WHEEL -->
     <joint name="left_wheel_joint" type="continuous">

Commit message: fix gazebo stl

File: agv_description/urdf/body.xacro (robot description, xacro)
@@ -9,12 +9,12 @@
         <origin xyz="0 0 0"/>
     </joint>
-    <joint name="gaizi_front_joint" type="fixed">
-        <parent link="base_link"/>
-        <child link="gaizi_front"/>
+    <joint name="cover_front_joint" type="fixed">
+        <parent link="base_link"/>
+        <child link="cover_front"/>
         <origin xyz="0 0 0"/>
     </joint>
-    <joint name="gaizi_back_joint" type="fixed">
-        <parent link="base_link"/>
-        <child link="gaizi_back"/>
+    <joint name="cover_back_joint" type="fixed">
+        <parent link="base_link"/>
+        <child link="cover_back"/>
         <origin xyz="0 0 0"/>
     </joint>
@@ -23,10 +23,9 @@
             <origin xyz="0 0 0" rpy="0 0 0" />
             <geometry>
-                <!-- <mesh filename="package://agv_description/meshes/chassis.stl" scale ="0.001 0.001 0.001"/> -->
-                <mesh filename="/home/cc/.gazebo/models/chassis.stl" scale ="0.001 0.001 0.001"/>
+                <mesh filename="file://$(find agv_description)/meshes/chassis.stl" scale ="0.001 0.001 0.001"/>
             </geometry>
             <material name="white"/>
         </visual>
-        <!-- <collision>
+        <collision>
             <origin xyz="0 0 0.4"/>
             <geometry>
@@ -36,13 +35,12 @@
         <xacro:inertial_box mass="10" x="1" y="0.52" z="0.7">
             <origin xyz="0 0 0.4" rpy="0 0 0"/>
-        </xacro:inertial_box> -->
-    </link>
-    <!-- gaizi_front -->
-    <link name="gaizi_front">
+        </xacro:inertial_box>
+    </link>
+    <!-- cover_front -->
+    <link name="cover_front">
         <visual>
             <origin xyz="0 0 0" rpy="0 0 0" />
             <geometry>
-                <!-- <mesh filename="package://agv_description/meshes/gaizi.stl" scale ="0.001 0.001 0.001"/> -->
-                <mesh filename="/home/cc/.gazebo/models/gaizi.stl" scale ="0.001 0.001 0.001"/>
+                <mesh filename="file://$(find agv_description)/meshes/cover.stl" scale ="0.001 0.001 0.001"/>
             </geometry>
             <material name="orange">
@@ -51,14 +49,13 @@
         </visual>
     </link>
-    <gazebo reference="gaizi_front">
+    <gazebo reference="cover_front">
 	    <material>Gazebo/Orange</material>
     </gazebo>
-    <!-- gaizi_back -->
-    <link name="gaizi_back">
+    <!-- cover_back -->
+    <link name="cover_back">
         <visual>
             <origin xyz="0 0 0" rpy="0 0 ${pi}" />
             <geometry>
-                <!-- <mesh filename="package://agv_description/meshes/gaizi.stl" scale ="0.001 0.001 0.001"/> -->
-                <mesh filename="/home/cc/.gazebo/models/gaizi.stl" scale ="0.001 0.001 0.001"/>
+                <mesh filename="file://$(find agv_description)/meshes/cover.stl" scale ="0.001 0.001 0.001"/>
             </geometry>
             <material name="orange">
@@ -67,5 +64,5 @@
         </visual>
     </link>
-    <gazebo reference="gaizi_back">
+    <gazebo reference="cover_back">
 	    <material>Gazebo/Orange</material>
     </gazebo>

Commit message: agv_look_color

File: agv_description/urdf/body.xacro (robot description, xacro)
@@ -27,5 +27,5 @@
             <material name="white"/>
         </visual>
-        <collision>
+        <!-- <collision>
             <origin xyz="0 0 0.4"/>
             <geometry>
@@ -35,5 +35,5 @@
         <xacro:inertial_box mass="10" x="1" y="0.52" z="0.7">
             <origin xyz="0 0 0.4" rpy="0 0 0"/>
-        </xacro:inertial_box>
+        </xacro:inertial_box> -->
     </link>
     <!-- cover_front -->
