Commit message: update urdf

File: agv_description/gazebo/body.xacro (robot description, xacro)
@@ -3,4 +3,10 @@
     <gazebo reference="chassis">
         <material>Gazebo/White</material>
+    </gazebo>
+    <gazebo reference="cover_front">
+	    <material>Gazebo/Orange</material>
+    </gazebo>
+    <gazebo reference="cover_back">
+	    <material>Gazebo/Orange</material>
     </gazebo>
     <gazebo reference="left_wheel">

File: agv_description/gazebo/lidar.xacro (robot description, xacro)
@@ -5,5 +5,5 @@
         <sensor name="laser" type="ray">
             <pose> 0 0 0 0 0 0 </pose>
-            <visualize>true</visualize>
+            <visualize>false</visualize>
             <update_rate>10</update_rate>
             <ray>

File: agv_description/urdf/body.xacro (robot description, xacro)
@@ -3,4 +3,11 @@
     <!-- BASE -->
     <link name="base_link"></link>
+    <!-- BASE FOOTPRINT -->
+    <joint name="base_footprint_joint" type="fixed">
+        <parent link="base_link"/>
+        <child link="base_footprint"/>
+        <origin xyz="0 0 0" rpy="0 0 0"/>
+    </joint>
+    <link name="base_footprint"></link>
     <!-- CHASSIS -->
     <joint name="chassis_joint" type="fixed">
@@ -9,4 +16,23 @@
         <origin xyz="0 0 0"/>
     </joint>
+    <link name="chassis">
+        <visual>
+            <origin xyz="0 0 0" rpy="0 0 0" />
+            <geometry>
+                <mesh filename="file://$(find agv_description)/meshes/chassis.stl" scale ="0.001 0.001 0.001"/>
+            </geometry>
+            <material name="white"/>
+        </visual>
+        <collision>
+            <origin xyz="0 0 0.4"/>
+            <geometry>
+                <box size="1 0.52 0.7"/>
+            </geometry>
+        </collision>
+        <xacro:inertial_box mass="10" x="1" y="0.52" z="0.7">
+            <origin xyz="0 0 0.4" rpy="0 0 0"/>
+        </xacro:inertial_box>
+    </link>
+    <!-- COVER FRONT -->
     <joint name="cover_front_joint" type="fixed">
         <parent link="base_link"/>
@@ -14,28 +40,4 @@
         <origin xyz="0 0 0"/>
     </joint>
-    <joint name="cover_back_joint" type="fixed">
-        <parent link="base_link"/>
-        <child link="cover_back"/>
-        <origin xyz="0 0 0"/>
-    </joint>
-    <link name="chassis">
-        <visual>
-            <origin xyz="0 0 0" rpy="0 0 0" />
-            <geometry>
-                <mesh filename="file://$(find agv_description)/meshes/chassis.stl" scale ="0.001 0.001 0.001"/>
-            </geometry>
-            <material name="white"/>
-        </visual>
-        <!-- <collision>
-            <origin xyz="0 0 0.4"/>
-            <geometry>
-                <box size="1 0.52 0.7"/>
-            </geometry>
-        </collision>
-        <xacro:inertial_box mass="10" x="1" y="0.52" z="0.7">
-            <origin xyz="0 0 0.4" rpy="0 0 0"/>
-        </xacro:inertial_box> -->
-    </link>
-    <!-- cover_front -->
     <link name="cover_front">
         <visual>
@@ -49,8 +51,10 @@
         </visual>
     </link>
-    <gazebo reference="cover_front">
-	    <material>Gazebo/Orange</material>
-    </gazebo>
-    <!-- cover_back -->
+    <!-- COVER BACK -->
+    <joint name="cover_back_joint" type="fixed">
+        <parent link="base_link"/>
+        <child link="cover_back"/>
+        <origin xyz="0 0 0"/>
+    </joint>
     <link name="cover_back">
         <visual>
@@ -64,7 +68,4 @@
         </visual>
     </link>
-    <gazebo reference="cover_back">
-	    <material>Gazebo/Orange</material>
-    </gazebo>
     <!-- LEFT WHEEL -->
     <joint name="left_wheel_joint" type="continuous">

Commit message: add nav

File: agv_description/gazebo/body.xacro (robot description, xacro)
@@ -11,28 +11,36 @@
     </gazebo>
     <gazebo reference="left_wheel">
-        <material>Gazebo/Blue</material>
+        <material>Gazebo/Gray</material>
+        <mu1 value="10000.0" />
+        <mu2 value="10000.0" />
+        <kp value="1e13" />
+        <kd value="1" />
     </gazebo>
     <gazebo reference="right_wheel">
-        <material>Gazebo/Blue</material>
+        <material>Gazebo/Gray</material>
+        <mu1 value="10000.0" />
+        <mu2 value="10000.0" />
+        <kp value="1e13" />
+        <kd value="1" />
     </gazebo>
     <gazebo reference="caster_left_front_wheel">
         <material>Gazebo/Black</material>
-        <mu1 value="0.005"/>
-        <mu2 value="0.005"/>
+        <mu1 value="0.0"/>
+        <mu2 value="0.0"/>
     </gazebo>
     <gazebo reference="caster_right_front_wheel">
         <material>Gazebo/Black</material>
-        <mu1 value="0.005"/>
-        <mu2 value="0.005"/>
+        <mu1 value="0.0"/>
+        <mu2 value="0.0"/>
     </gazebo>
     <gazebo reference="caster_left_back_wheel">
         <material>Gazebo/Black</material>
-        <mu1 value="0.005"/>
-        <mu2 value="0.005"/>
+        <mu1 value="0.0"/>
+        <mu2 value="0.0"/>
     </gazebo>
     <gazebo reference="caster_right_back_wheel">
         <material>Gazebo/Black</material>
-        <mu1 value="0.005"/>
-        <mu2 value="0.005"/>
+        <mu1 value="0.0"/>
+        <mu2 value="0.0"/>
     </gazebo>
 </robot>

File: agv_description/urdf/body.xacro (robot description, xacro)
@@ -74,4 +74,6 @@
         <origin xyz="0 0.192 0.075" rpy="-${pi/2} 0 0" />
         <axis xyz="0 0 1"/>
+        <limit effort="1000.0" lower="-1e50" upper="1e50" velocity="30"/>
+        <dynamics damping="0.0" friction="0.0"/>
     </joint>
     <link name="left_wheel">
@@ -84,5 +86,6 @@
         <collision>
             <geometry>
-                <cylinder radius="0.075" length="0.05"/>
+                <!-- <cylinder radius="0.075" length="0.05"/> -->
+                <sphere radius="0.075"/>
             </geometry>
         </collision>
@@ -97,4 +100,6 @@
         <origin xyz="0 -0.192 0.075" rpy="${pi/2} 0 0" />
         <axis xyz="0 0 -1"/>
+        <limit effort="1000.0" lower="-1e50" upper="1e50" velocity="30"/>
+        <dynamics damping="0.0" friction="0.0"/>
     </joint>
     <link name="right_wheel">
@@ -107,5 +112,6 @@
         <collision>
             <geometry>
-                <cylinder radius="0.075" length="0.05"/>
+                <!-- <cylinder radius="0.075" length="0.05"/> -->
+                <sphere radius="0.075"/>
             </geometry>
         </collision>
@@ -132,7 +138,7 @@
             </geometry>
         </collision>
-        <xacro:inertial_sphere mass="1" radius="0.06">
-            <origin xyz="0 0 0" rpy="0 0 0"/>
-        </xacro:inertial_sphere>
+        <!-- <xacro:inertial_sphere mass="1" radius="0.06">
+            <origin xyz="0 0 0" rpy="0 0 0"/>
+        </xacro:inertial_sphere> -->
     </link>
     <joint name="caster_right_front_wheel_joint" type="fixed">
@@ -153,7 +159,7 @@
             </geometry>
         </collision>
-        <xacro:inertial_sphere mass="1" radius="0.06">
-            <origin xyz="0 0 0" rpy="0 0 0"/>
-        </xacro:inertial_sphere>
+        <!-- <xacro:inertial_sphere mass="1" radius="0.06">
+            <origin xyz="0 0 0" rpy="0 0 0"/>
+        </xacro:inertial_sphere> -->
     </link>
     <joint name="caster_left_back_wheel_joint" type="fixed">
@@ -174,7 +180,7 @@
             </geometry>
         </collision>
-        <xacro:inertial_sphere mass="1" radius="0.06">
-            <origin xyz="0 0 0" rpy="0 0 0"/>
-        </xacro:inertial_sphere>
+        <!-- <xacro:inertial_sphere mass="1" radius="0.06">
+            <origin xyz="0 0 0" rpy="0 0 0"/>
+        </xacro:inertial_sphere> -->
     </link>
     <joint name="caster_right_back_wheel_joint" type="fixed">
@@ -195,7 +201,7 @@
             </geometry>
         </collision>
-        <xacro:inertial_sphere mass="1" radius="0.06">
-            <origin xyz="0 0 0" rpy="0 0 0"/>
-        </xacro:inertial_sphere>
+        <!-- <xacro:inertial_sphere mass="1" radius="0.06">
+            <origin xyz="0 0 0" rpy="0 0 0"/>
+        </xacro:inertial_sphere> -->
     </link>
 </robot>
